File: PCB/raspberrrypi_hat/M590.sch (KiCad schematic (older format))
At the start: 12 parts, among them J4 Micro_SIM_Card, U2 NeowayM590

Commit message: PCB: Change RPi header + add Micro SIM socket. Starting placement
Parts:
- C1, C3, C4: footprint (none) -> Capacitors_SMD:C_1206_HandSoldering
- J4: footprint (none) -> project_footprints:MicroSIMSocket
Changed lines of the file:
@@
 F 0 "J4" H 8700 3750 50  0000 R CNN
 F 1 "Micro_SIM_Card" H 8400 3650 50  0000 L CNN
-F 2 "" H 8800 3600 50  0000 C CNN
+F 2 "project_footprints:MicroSIMSocket" H 8800 3600 50  0001 C CNN
 F 3 "" H 8750 3250 50  0000 C CNN
 	1    8800 3250
@@
 	2650 6750 2650 6900
 Wire Wire Line
-	2150 6200 2150 6350
-Wire Wire Line
-	2150 6350 2150 6450
+	2150 6200 2150 6450
 Wire Wire Line
 	2150 5800 2150 5900
 $Comp
-L GND #PWR14
+L GND #PWR08
 U 1 1 595187AA
 P 2650 6900
-F 0 "#PWR14" H 2650 6650 50  0001 C CNN
+F 0 "#PWR08" H 2650 6650 50  0001 C CNN
 F 1 "GND" H 2650 6750 50  0000 C CNN
 F 2 "" H 2650 6900 50  0001 C CNN
@@
 $EndComp
 $Comp
-L GND #PWR9
+L GND #PWR09
 U 1 1 595187F4
 P 3900 3800
-F 0 "#PWR9" H 3900 3550 50  0001 C CNN
+F 0 "#PWR09" H 3900 3550 50  0001 C CNN
 F 1 "GND" H 3900 3650 50  0000 C CNN
 F 2 "" H 3900 3800 50  0001 C CNN
@@
 P5V
 $Comp
-L GND #PWR7
+L GND #PWR010
 U 1 1 5952C140
 P 1650 1200
-F 0 "#PWR7" H 1650 950 50  0001 C CNN
+F 0 "#PWR010" H 1650 950 50  0001 C CNN
 F 1 "GND" H 1650 1050 50  0000 C CNN
 F 2 "" H 1650 1200 50  0001 C CNN
@@
 	4900 2850 5250 2850
 Wire Wire Line
-	4900 2550 4900 2850
-Wire Wire Line
-	4900 2850 4900 3800
-Wire Wire Line
-	6900 2550 6900 3050
-Wire Wire Line
-	6900 3050 6900 3800
-$Comp
-L GND #PWR12
+	4900 2550 4900 3800
+Wire Wire Line
+	6900 2550 6900 3800
+$Comp
+L GND #PWR011
 U 1 1 5952C301
 P 8150 3800
-F 0 "#PWR12" H 8150 3550 50  0001 C CNN
+F 0 "#PWR011" H 8150 3550 50  0001 C CNN
 F 1 "GND" H 8150 3650 50  0000 C CNN
 F 2 "" H 8150 3800 50  0001 C CNN
@@
 $EndComp
 $Comp
-L GND #PWR10
+L GND #PWR012
 U 1 1 5952C323
 P 4900 3800
-F 0 "#PWR10" H 4900 3550 50  0001 C CNN
+F 0 "#PWR012" H 4900 3550 50  0001 C CNN
 F 1 "GND" H 4900 3650 50  0000 C CNN
 F 2 "" H 4900 3800 50  0001 C CNN
@@
 $EndComp
 Wire Wire Line
-	4250 2650 5100 2650
-Wire Wire Line
-	5100 2650 5250 2650
+	4250 2650 5250 2650
 Wire Wire Line
 	5250 2750 5100 2750
@@
 	8150 3250 8150 3800
 $Comp
-L GND #PWR11
+L GND #PWR013
 U 1 1 59540978
 P 6900 3800
-F 0 "#PWR11" H 6900 3550 50  0001 C CNN
+F 0 "#PWR013" H 6900 3550 50  0001 C CNN
 F 1 "GND" H 6900 3650 50  0000 C CNN
 F 2 "" H 6900 3800 50  0001 C CNN
@@
 $EndComp
 Wire Wire Line
-	6550 3150 7300 3150
-Wire Wire Line
-	7300 3150 7850 3150
+	6550 3150 7850 3150
 Wire Wire Line
 	7850 3150 7850 2950
@@
 	8050 3150 8300 3150
 Wire Wire Line
-	6550 3450 7800 3450
-Wire Wire Line
-	7800 3450 8300 3450
+	6550 3450 8300 3450
 Connection ~ 6900 3050
 Connection ~ 4900 2850
@@
 F 0 "C3" H 2675 6700 50  0000 L CNN
 F 1 "0.1µF" H 2675 6500 50  0000 L CNN
-F 2 "" H 2688 6450 50  0001 C CNN
+F 2 "Capacitors_SMD:C_1206_HandSoldering" H 2688 6450 50  0001 C CNN
 F 3 "" H 2650 6600 50  0001 C CNN
 	1    2650 6600
@@
 F 0 "C4" H 3175 6700 50  0000 L CNN
 F 1 "100pF" H 3175 6500 50  0000 L CNN
-F 2 "" H 3188 6450 50  0001 C CNN
+F 2 "Capacitors_SMD:C_1206_HandSoldering" H 3188 6450 50  0001 C CNN
 F 3 "" H 3150 6600 50  0001 C CNN
 	1    3150 6600
@@
 	2150 6750 2150 6900
 $Comp
-L GND #PWR13
+L GND #PWR014
 U 1 1 5954184B
 P 2150 6900
-F 0 "#PWR13" H 2150 6650 50  0001 C CNN
+F 0 "#PWR014" H 2150 6650 50  0001 C CNN
 F 1 "GND" H 2150 6750 50  0000 C CNN
 F 2 "" H 2150 6900 50  0001 C CNN
@@
 	3150 6750 3150 6900
 $Comp
-L GND #PWR15
+L GND #PWR015
 U 1 1 5954186F
 P 3150 6900
-F 0 "#PWR15" H 3150 6650 50  0001 C CNN
+F 0 "#PWR015" H 3150 6650 50  0001 C CNN
 F 1 "GND" H 3150 6750 50  0000 C CNN
 F 2 "" H 3150 6900 50  0001 C CNN
@@
 $EndComp
 Wire Wire Line
-	2150 6350 2650 6350
-Wire Wire Line
-	2650 6350 3150 6350
-Wire Wire Line
-	3150 6350 3850 6350
+	2150 6350 3850 6350
 Wire Wire Line
 	2650 6350 2650 6450
@@
 $EndComp
 Wire Wire Line
-	1850 3450 2100 3450
-Wire Wire Line
-	2100 3450 2400 3450
+	1850 3450 2400 3450
 $Comp
 L C C1
@@
 F 0 "C1" H 2125 3800 50  0000 L CNN
 F 1 "100pF" H 2125 3600 50  0000 L CNN
-F 2 "" H 2138 3550 50  0001 C CNN
+F 2 "Capacitors_SMD:C_1206_HandSoldering" H 2138 3550 50  0001 C CNN
 F 3 "" H 2100 3700 50  0001 C CNN
 	1    2100 3700
@@
 	2100 3850 2100 4000
 $Comp
-L GND #PWR8
+L GND #PWR016
 U 1 1 5954200E
 P 2100 4000
-F 0 "#PWR8" H 2100 3750 50  0001 C CNN
+F 0 "#PWR016" H 2100 3750 50  0001 C CNN
 F 1 "GND" H 2100 3850 50  0000 C CNN
 F 2 "" H 2100 4000 50  0001 C CNN
@@
 	2100 3550 2100 3450
 $Comp
-L GND #PWR?
+L GND #PWR017
 U 1 1 595571B7
 P 1650 1900
-F 0 "#PWR?" H 1650 1650 50  0001 C CNN
+F 0 "#PWR017" H 1650 1650 50  0001 C CNN
 F 1 "GND" H 1650 1750 50  0000 C CNN
 F 2 "" H 1650 1900 50  0001 C CNN

Commit message: Fix TX/RX serial resistor short-cut by adding mTX/mRX in M590 module sheet
Connections:
- net RXD: no longer C1.1, R10.1, U2.7 (RXD)
- net TXD: no longer R9.1, U2.8 (TXD)
- new net mRXD: C1.1, R10.1, U2.7 (RXD)
- new net mTXD: R9.1, U2.8 (TXD)
Changed lines of the file:
@@
 BOOT
 Text Label 2400 3450 2    60   ~ 0
-RXD
+mRXD
 Text Label 2400 3300 2    60   ~ 0
-TXD
+mTXD
 Wire Wire Line
 	6550 2550 6900 2550
@@
 	5250 3250 4250 3250
 Text Label 4250 3150 0    60   ~ 0
-RXD
+mRXD
 Text Label 4250 3250 0    60   ~ 0
-TXD
+mTXD
 Wire Wire Line
 	5250 3450 4250 3450
