File: PCB/raspberrrypi_hat/M590.sch (KiCad schematic (older format))
At the start: 12 parts, among them J4 Micro_SIM_Card, U2 NeowayM590

Commit message: Change LED footprint to 1206 HandSoldering
Parts:
- D1: footprint LEDs:LED_0603 -> LEDs:LED_1206_HandSoldering
Changed lines of the file:
@@
 F 0 "D1" H 3900 3650 50  0000 C CNN
 F 1 "LED" H 3900 3450 50  0000 C CNN
-F 2 "LEDs:LED_0603" H 3900 3550 50  0001 C CNN
+F 2 "LEDs:LED_1206_HandSoldering" H 3900 3550 50  0001 C CNN
 F 3 "" H 3900 3550 50  0001 C CNN
 	1    3900 3550

Commit message: Fix #5 Change R9/R10 to 220R
Parts:
- R10, R9: value 200 -> 220
Changed lines of the file:
@@
 P 1700 3450
 F 0 "R10" V 1780 3450 50  0000 C CNN
-F 1 "200" V 1700 3450 50  0000 C CNN
+F 1 "220" V 1700 3450 50  0000 C CNN
 F 2 "Resistors_SMD:R_1206_HandSoldering" V 1630 3450 50  0001 C CNN
 F 3 "" H 1700 3450 50  0001 C CNN
@@
 P 1700 3300
 F 0 "R9" V 1780 3300 50  0000 C CNN
-F 1 "200" V 1700 3300 50  0000 C CNN
+F 1 "220" V 1700 3300 50  0000 C CNN
 F 2 "Resistors_SMD:R_1206_HandSoldering" V 1630 3300 50  0001 C CNN
 F 3 "" H 1700 3300 50  0001 C CNN
