File: PCB/raspberrrypi_hat/raspberrrypi_hat.kicad_pcb (KiCad board)
At the start: 4 copper layers, 65 x 56 mm, 30 parts, among them J1 40HAT, J2 CONN_02X02, J3 CONN_01X02, J4 Micro_SIM_Card, Q1 DMG2305UX, Q2 DMMT5401, U1 CAT24C32, U2 NeowayM590

Commit message: Mark the project with Creative Commons by-nc-nd license
Parts:
- added G***: LOGO, project_footprints:LOGO_CC-by-nc-nd-eu, B.Cu at (89.0, 89.7)

Commit message: PCB: Add small CC-by-nc-nd license logo to PCB front side
Parts:
- added G***: LOGO, project_footprints:LOGO_CC-by-nc-nd-small, F.Cu at (140.1, 80.1)
